File: Hardware/Kicad Project/ArduinoProMicroUSB/ArduinoProMicroUSB.sch (KiCad schematic (older format))
At the start: 45 parts, among them J1 Battery, J3 Display FPC, Q1 MMBT3904, SW1 SW_Push, SW2 SW_Push, SW3 SW_Push, SW4 SW_Push, U1 RV-3028-C7, U2 MIC5219, U3 USB-AB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

Commit message: rev 0.1
Other:
- moved on the sheet: C1, C10, C11, C12, C13, C2, C3, C4, C5, C6, C7, C8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

Commit message: rev 0.2
Parts:
- removed SJ1: Closed for 5V Board, Downloads:Jumper, symbol ArduinoProMicroUSB-eagle-import:SOLDERJUMPERNC
- C8: value 10nF -> 100nF
Connections:
- wire segments 196 -> 191
- no-connect marks 12 -> 13
Other:
- moved on the sheet: C1, C13, C2, C3, C4, D1, F1, LED1, R2, U2
