File: Hardware/Kicad Project/ArduinoProMicroUSB/ArduinoProMicroUSB.sch (KiCad schematic (older format))
At the start: 44 parts, among them J1 Battery, J3 Display FPC, Q1 MMBT3904, SW1 SW_Push, SW2 SW_Push, SW3 SW_Push, SW4 SW_Push, U1 RV-3028-C7, U2 MIC5219, U3 USB-AB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

Commit message: rev 0,2
Other:
- note added: "?"
- moved on the sheet: R12, R13, R14, R15, R5, R7, SW1, SW2, SW3, SW4

Commit message: updated schematic
Parts:
- removed J1: Battery, Connector_PinSocket_2.54mm:PinSocket_1x02_P2.54mm_Vertical, symbol Connector:Conn_01x02_Female
- added C14, C15, C16, C9: 100pF, Capacitor_SMD:C_0603_1608Metric, symbol ArduinoProMicroUSB-eagle-import:CAP0603-CAP
- added D4: PRTR5V0U2X,215, SOT143B, symbol ArduinoProMicroUSB-eagle-import:PRTR5V0U2X,215
- added J1: Conn2, symbol ArduinoProMicroUSB-eagle-import:Conn2
- U2: value MIC5219 -> V_REG_LDOSMD; footprint Downloads:SOT23-5 -> (none)
- U3: footprint Connectors:USB-AB-MICRO-SMD -> (none)
Connections:
- wire segments 191 -> 226
- no-connect marks 12 -> 11
Other:
- note removed: "?"
- moved on the sheet: C1, C13, C2, C3, C4, D1, F1, LED1, R12, R13, R14, R15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

Commit message: updated schematic
Parts:
- removed C1, C2: 10uF, Capacitors:EIA3216, symbol ArduinoProMicroUSB-eagle-import:CAP_POL1206
- removed C13: 470pF, Capacitor_SMD:C_0603_1608Metric, symbol ArduinoProMicroUSB-eagle-import:CAP0603-CAP
- removed C3: 1uF, Capacitor_SMD:C_0603_1608Metric, symbol ArduinoProMicroUSB-eagle-import:CAP0603-CAP
- removed C4: 0.1uF, Capacitor_SMD:C_0603_1608Metric, symbol ArduinoProMicroUSB-eagle-import:CAP0603-CAP
- removed C8: 100nF, Capacitor_SMD:C_0603_1608Metric, symbol ArduinoProMicroUSB-eagle-import:CAP0603-CAP
- removed D1: DIODESOD, Diode_SMD:D_SOD-123, symbol ArduinoProMicroUSB-eagle-import:DIODESOD
- removed F1: 500mA, Fuse:Fuse_1812_4532Metric, symbol Device:Fuse_Small
- removed LED1: Red, Diode_SMD:D_0603_1608Metric, symbol ArduinoProMicroUSB-eagle-import:LED0603
- removed R2: 1K, Resistor_SMD:R_0603_1608Metric, symbol ArduinoProMicroUSB-eagle-import:RESISTOR0603-RES
- removed RN2: R_Pack04, Resistor_SMD:R_Array_Concave_4x0603, symbol Device:R_Pack04
- removed U2: V_REG_LDOSMD, symbol ArduinoProMicroUSB-eagle-import:V_REG_LDOSMD
- added C1, C2: 100nF, symbol Device:C
- added C17: 4.7uF, Capacitor_SMD:C_0603_1608Metric, symbol ArduinoProMicroUSB-eagle-import:CAP0603-CAP
- added C18: 10uF, Capacitor_SMD:C_0603_1608Metric, symbol ArduinoProMicroUSB-eagle-import:CAP0603-CAP
- added L1: 2.2uH, symbol pspice:INDUCTOR
- added R10, R2: 6k, symbol Device:R
- added R16: 267k, symbol Device:R
- added U4: TPS62840DLCR, SON50P200X150X100-8N, symbol ArduinoProMicroUSB-eagle-import:TPS62840DLCR
- J3: value Display FPC -> FPC
- R9: value 10K -> R; footprint Resistor_SMD:R_0603_1608Metric -> (none)
Connections:
- net labels added: INT
- net labels removed: 32K, CS, DC, EVI, RAW, RST, SQW, TFT_DIN, TFT_SCK
- wire segments 226 -> 224
- no-connect marks 11 -> 13
Other:
- note added: "Buttons"
- note added: "CS"
- note added: "DC"
- note added: "DIN"
- note added: "GND"
- note added: "LEDA"
- note added: "LEDK"
- note added: "MCU"
- note added: "Power(BAT,USB,REGULATOR)"
- note added: "RST"
- note added: "RTC Clock"
- note added: "SCK"
- note added: "VDD"
- note removed: "Battery"
- note removed: "Clock"
- note removed: "Connections"
- note removed: "Microcontroller"
- note removed: "https://www.waveshare.com/w/upload/0/0c/1.3inch_LCD_Module_Schematic.pdf"
- moved on the sheet: C10, C11, C12, C14, C15, C16, C5, C6, C7, C9, D2, D3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

Commit message: pdf
Parts:
- added TP1, TP2, TP3, TP4, TP5: TestPoint, symbol Connector:TestPoint
Connections:
- net D2: now also TP5.1
- net D3: now also TP4.1
- net MISO: now also TP1.1
- net MOSI: now also TP2.1
- net SCK: now also TP3.1
Changed lines of the file:
@@
 Wire Wire Line
 	12285 1930 14440 1930
+$Comp
+L Connector:TestPoint TP4
+U 1 1 61D5E7DE
+P 12790 1430
+F 0 "TP4" V 12685 1685 50  0000 C CNN
+F 1 "TestPoint" V 12860 1610 50  0001 C CNN
+F 2 "" H 12990 1430 50  0001 C CNN
+F 3 "~" H 12990 1430 50  0001 C CNN
+	1    12790 1430
+	0    -1   -1   0
+$EndComp
+$Comp
+L Connector:TestPoint TP5
+U 1 1 61D70684
+P 12790 1530
+F 0 "TP5" V 12885 1785 50  0000 C CNN
+F 1 "TestPoint" V 12725 1700 50  0001 C CNN
+F 2 "" H 12990 1530 50  0001 C CNN
+F 3 "~" H 12990 1530 50  0001 C CNN
+	1    12790 1530
+	0    -1   -1   0
+$EndComp
+$Comp
+L Connector:TestPoint TP3
+U 1 1 61D85099
+P 12285 6360
+F 0 "TP3" V 12275 6680 50  0000 R CNN
+F 1 "TestPoint" V 12389 6432 50  0001 C CNN
+F 2 "" H 12485 6360 50  0001 C CNN
+F 3 "~" H 12485 6360 50  0001 C CNN
+	1    12285 6360
+	0    -1   -1   0
+$EndComp
+$Comp
+L Connector:TestPoint TP2
+U 1 1 61D9428D
+P 12175 6460
+F 0 "TP2" V 12085 6655 50  0000 R CNN
+F 1 "TestPoint" V 12279 6532 50  0001 C CNN
+F 2 "" H 12375 6460 50  0001 C CNN
+F 3 "~" H 12375 6460 50  0001 C CNN
+	1    12175 6460
+	0    -1   -1   0
+$EndComp
+$Comp
+L Connector:TestPoint TP1
+U 1 1 61DA3362
+P 12070 6260
+F 0 "TP1" V 12065 6490 50  0000 C CNN
+F 1 "TestPoint" H 12055 6805 50  0001 C CNN
+F 2 "" H 12270 6260 50  0001 C CNN
+F 3 "~" H 12270 6260 50  0001 C CNN
+	1    12070 6260
+	0    -1   -1   0
+$EndComp
+Connection ~ 12070 6260
+Connection ~ 12175 6460
+Connection ~ 12285 6360
 $EndSCHEMATC

Commit message: rev 0.4
Parts:
- added TP6, TP7: TestPoint, TestPoint:TestPoint_Pad_1.0x1.0mm, symbol Connector:TestPoint
- C1, C2: footprint (none) -> Capacitor_SMD:C_0603_1608Metric
- D4: footprint SOT143B -> Downloads:SOT143B
- J1: footprint (none) -> Downloads:1X02
- L1: footprint (none) -> Inductor_SMD:L_0603_1608Metric
- R10, R16, R2, R9: footprint (none) -> Resistor_SMD:R_0603_1608Metric
- TP1, TP2, TP3, TP4, TP5: footprint (none) -> TestPoint:TestPoint_Pad_1.0x1.0mm
- U3: footprint (none) -> Downloads:USB-AB-MICRO-SMD
- U4: footprint SON50P200X150X100-8N -> Downloads:SON50P200X150X100-8N
Connections:
- net GND: now also TP6.1
- net at J1.1: now also TP7.1
- no-connect marks 13 -> 15
Other:
- note added: "Battery"
- note added: "Regulator"
- note added: "USB"
- note removed: "Power(BAT,USB,REGULATOR)"
- moved on the sheet: C1, C10, C11, C12, C14, C15, C16, C17, C18, C2, C5, C6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

Commit message: working on pcb
Parts:
- C1, C10, C11, C12, C14, C15, C16, C17, C18, C2, C5, C6, C7, C9: footprint Capacitor_SMD:C_0603_1608Metric -> Downloads:0603
- L1: footprint Inductor_SMD:L_0603_1608Metric -> Downloads:0603
- R1, R10, R11, R12, R13, R14, R15, R16, R2, R3, R4, R5, R6, R7, R8, R9: footprint Resistor_SMD:R_0603_1608Metric -> Downloads:0603
- SW1, SW2, SW3, SW4: footprint Downloads:FSMRACD -> Downloads:Panasonic-EVP-AKE31A-MFG
- U5: footprint Package_QFP:TQFP-44_10x10mm_P0.8mm -> Downloads:QFN50P700X700X100-45N
Connections:
- net D12: now also J3.8 (Pin_8), TP1.1
- net MISO: no longer J3.8 (Pin_8), TP1.1
- no-connect marks 15 -> 13
