File: Hardware/Kicad Project/ArduinoProMicroUSB/ArduinoProMicroUSB.sch (KiCad schematic (older format))
At the start: 53 parts, among them J1 Conn2, J3 FPC, Q1 MMBT3904, SW1 SW_Push, SW2 SW_Push, SW3 SW_Push, SW4 SW_Push, U1 RV-3028-C7, U3 USB-AB, U4 TPS62840DLCR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

Commit message: schematic checking
Connections:
- net A3: no longer names the net of U5.39 (PF4(ADC4))
- net A4: no longer names the net of U5.40 (PF1(ADC1))
- net A5: no longer names the net of U5.41 (PF0(ADC0))
- no-connect marks 13 -> 15
Changed lines of the file:
@@
 Text Label 6320 3370 0    70   ~ 0
 D2
-Text Label 6320 2570 0    70   ~ 0
-A3
-Text Label 6320 2670 0    70   ~ 0
-A4
-Text Label 6320 2770 0    70   ~ 0
-A5
 Text Label 6320 3970 0    70   ~ 0
 D8
@@
 	1    0    0    -1
 $EndComp
+NoConn ~ 6555 4470
+NoConn ~ 6555 4870
 $EndSCHEMATC
