File: Hardware/Kicad Project/ArduinoProMicroUSB/ArduinoProMicroUSB.kicad_pcb (KiCad board)
At the start: 4 copper layers, 32 x 26.4 mm, 41 parts, among them J1 Battery, J3 Display FPC, Q1 MMBT3904, U1 RV-3028-C7, U2 MIC5219, U3 USB-AB, U5 ATMEGA32U4QFN, Y1 16MHz

Commit message: rev 0.1
Parts:
- added 3.3V: TestPoint_THTPad_2.0x2.0mm_Drill1.0mm, TestPoint:TestPoint_THTPad_2.0x2.0mm_Drill1.0mm, F.Cu at (144.9, 77.9)
- moved SJ1 8.28 mm to (128.8, 77.3)
- moved C1 4.66 mm to (135.2, 76.7)
- moved J1 4.33 mm to (131.7, 95.6)
- moved C2 4.08 mm to (138.8, 78.7)
- moved C4 3.96 mm to (136.9, 79.5)
- moved U3 3.86 mm to (137.9, 97.4)
- moved U2 3.61 mm to (133.7, 79.5)
- moved R7 3.41 mm to (138.3, 92.2)
- moved R5 3.36 mm to (137.0, 92.2)
- moved D1 3.32 mm to (131.8, 85.7)
- moved F1 2.78 mm to (132.1, 91.3)
- moved C13 2.18 mm to (133.0, 82.1), turned to 180 degrees
- moved R12 0.99 mm to (136.8, 82.1)
- moved R3 0.98 mm to (155.8, 79.8)
- moved C8 0.96 mm to (150.3, 97.9)
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Routing:
- net Net-(D1-Pad2): track 3.86 -> 13.1 mm
- net 3.3V: track 66.3 -> 58.9 mm, vias 19 -> 21
- net GND: track 41.5 -> 46.9 mm, vias 19 -> 22
- net /RAW: track 7.05 -> 10.9 mm
- net /D+: track 13.0 -> 14.6 mm
- net Net-(C13-Pad1): track 1.36 -> 2.93 mm
- net /D-: track 13.7 -> 15.1 mm
- net /D5: track 25.0 -> 26.0 mm
- net Net-(R7-Pad2): track 2.88 -> 1.94 mm
- net Net-(R5-Pad2): track 2.60 -> 1.90 mm
- net Net-(R4-Pad2): track 2.99 -> 2.48 mm
Other:
- board size 32 x 26.4 mm -> 28.3 x 24.8 mm

Commit message: rev 0.1
Parts:
- removed J1: Battery, Connector_PinSocket_2.54mm:PinSocket_1x02_P2.54mm_Vertical
- added -Battery+: TestPoint_THTPad_1.5x1.5mm_Drill0.7mm, TestPoint:TestPoint_THTPad_1.5x1.5mm_Drill0.7mm, F.Cu at (131.7, 97.6)
- added REF**: TestPoint_THTPad_1.5x1.5mm_Drill0.7mm, TestPoint:TestPoint_THTPad_1.5x1.5mm_Drill0.7mm, F.Cu at (131.7, 95.5)
- moved R5 1.02 mm to (136.0, 91.9)
- moved R7 0.87 mm to (137.5, 91.9)
- moved U1 0.82 mm to (154.1, 94.9)
- moved RN2 0.75 mm to (150.8, 94.9)
- moved C8 0.55 mm to (150.8, 97.7)
- moved U3 0.27 mm to (137.8, 97.7)
- moved R9 0.16 mm to (152.1, 91.6)
- renumbered U2 to UE
Routing:
- net 3.3V: track 58.9 -> 55.5 mm, vias 21 -> 20
- net Net-(R9-Pad1): track 4.13 -> 0.79 mm
- net GND: track 46.9 -> 44.1 mm
- net VCC: track 27.6 -> 28.9 mm
- net /D-: track 15.1 -> 14.0 mm
- net /D12: track 15.8 -> 16.9 mm
- net Net-(R5-Pad2): track 1.90 -> 2.84 mm
- net /D2: track 15.9 -> 15.0 mm
- net /D+: track 14.6 -> 13.8 mm
Other:
- board size 28.3 x 24.8 mm -> 28.3 x 25.2 mm

Commit message: rev 0.1
Parts:
- added 3.3: TestPoint_THTPad_1.5x1.5mm_Drill0.7mm, TestPoint:TestPoint_THTPad_1.5x1.5mm_Drill0.7mm, F.Cu at (128.9, 88.5)
- added CS: TestPoint_THTPad_1.5x1.5mm_Drill0.7mm, TestPoint:TestPoint_THTPad_1.5x1.5mm_Drill0.7mm, F.Cu at (128.9, 81.7)
- added GND: TestPoint_THTPad_1.5x1.5mm_Drill0.7mm, TestPoint:TestPoint_THTPad_1.5x1.5mm_Drill0.7mm, F.Cu at (128.9, 93.1)
- added MOSI: TestPoint_THTPad_1.5x1.5mm_Drill0.7mm, TestPoint:TestPoint_THTPad_1.5x1.5mm_Drill0.7mm, F.Cu at (128.9, 79.2)
- added SCK: TestPoint_THTPad_1.5x1.5mm_Drill0.7mm, TestPoint:TestPoint_THTPad_1.5x1.5mm_Drill0.7mm, F.Cu at (128.9, 76.8)
- added SCL: TestPoint_THTPad_1.5x1.5mm_Drill0.7mm, TestPoint:TestPoint_THTPad_1.5x1.5mm_Drill0.7mm, F.Cu at (128.9, 83.9)
- added SDA: TestPoint_THTPad_1.5x1.5mm_Drill0.7mm, TestPoint:TestPoint_THTPad_1.5x1.5mm_Drill0.7mm, F.Cu at (128.9, 86.2)
- added VCC: TestPoint_THTPad_1.5x1.5mm_Drill0.7mm, TestPoint:TestPoint_THTPad_1.5x1.5mm_Drill0.7mm, F.Cu at (128.9, 90.8)
- moved J3 6.29 mm to (132.8, 82.4)
- moved REF** 2.77 mm to (128.9, 95.4)
- moved +Battery- 2.77 mm to (128.9, 97.7)
- moved SJ1 0.27 mm to (129.0, 77.3)
- moved C1 0.26 mm to (135.5, 76.7)
- moved C10 0.25 mm to (143.0, 77.7)
- moved C13 0.25 mm to (133.3, 82.1)
- moved C2 0.25 mm to (139.0, 78.7)
- moved C4 0.25 mm to (137.2, 79.5)
- moved C5 0.25 mm to (147.6, 94.0)
- moved C7 0.25 mm to (155.3, 77.4)
- moved D2 0.25 mm to (153.2, 88.7)
- moved D3 0.25 mm to (137.0, 89.2)
- moved LED1 0.25 mm to (147.9, 77.7)
- moved Q1 0.25 mm to (152.1, 79.6)
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- renumbered -Battery+ to +Battery-
Routing:
- net GND: track 44.1 -> 70.5 mm, vias 22 -> 23
- net /D3: track 21.0 -> 45.6 mm, vias 0 -> 1
- net /D2: track 15.0 -> 38.8 mm
- net /LEDK: track 1.04 -> 19.9 mm
- net /SCK: track 9.28 -> 27.0 mm
- net /MOSI: track 9.17 -> 25.1 mm
- net 3.3V: track 55.5 -> 71.0 mm, vias 20 -> 19
- net /CS: track 12.2 -> 25.8 mm
- net VCC: track 28.9 -> 40.8 mm, vias 1 -> 0
- net /D4: track 21.1 -> 16.5 mm
- net Net-(R9-Pad1): track 0.79 -> 4.77 mm
- net /D5: track 26.0 -> 24.3 mm
- net /32K: track 18.7 -> 19.6 mm
Other:
- board size 28.3 x 25.2 mm -> 31.1 x 26 mm

Commit message: rev 0.2
Parts:
- moved D2 1.53 mm to (154.7, 88.8)
- moved R6 1.50 mm to (153.2, 88.8)
- moved U1 0.80 mm to (154.5, 94.2)
- moved 3.3V 0.33 mm to (145.4, 77.7)
- moved SJ1 0.18 mm to (129.0, 77.2)
- moved R4 0.16 mm to (141.7, 93.3)
- moved Q1 0.15 mm to (152.1, 79.8)
- moved Y1 0.14 mm to (146.1, 96.7)
- moved LED1 0.10 mm to (147.9, 77.6)
- moved C3 0.10 mm to (141.6, 77.6)
- moved R9 0.10 mm to (152.2, 91.6)
- moved C10 0.10 mm to (143.0, 77.6)
- moved R2 0.10 mm to (149.4, 77.6)
Routing:
- net 3.3V: track 71.0 -> 56.3 mm, vias 19 -> 10
- net GND: track 70.5 -> 67.1 mm, vias 23 -> 19
- net VCC: track 40.8 -> 43.4 mm
- net Net-(R6-Pad1): track 6.02 -> 4.49 mm
- net /32K: track 19.6 -> 18.3 mm
- net /D12: track 16.9 -> 15.9 mm
- net Net-(R9-Pad1): track 4.77 -> 4.24 mm

Commit message: gif
Parts:
- moved C1 0.05 mm to (135.5, 76.7)
Changed lines of the file:
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@@
   )
   (module Capacitors:EIA3216 (layer F.Cu)
-    (at 135.46074 76.708 180)
+    (at 135.46074 76.6572 180)
     (descr "GENERIC EIA 3216 (1206) POLARIZED TANTALUM CAPACITOR")
     (tags "GENERIC EIA 3216 (1206) POLARIZED TANTALUM CAPACITOR")

Commit message: rev 0.2
Parts:
- renumbered UE to U2

Commit message: rev 0.2
Parts:
- removed +Battery-: TestPoint_THTPad_1.5x1.5mm_Drill0.7mm, TestPoint:TestPoint_THTPad_1.5x1.5mm_Drill0.7mm
- removed the REF** at (128.9, 95.4)
- removed SJ1: Closed for 5V Board, Downloads:Jumper
- added REF**: MountingHole_2.1mm, MountingHole:MountingHole_2.1mm, F.Cu at (156.3, 75.7)
- added REF**: MountingHole_2.1mm, MountingHole:MountingHole_2.1mm, F.Cu at (127.8, 75.7)
- added REF**: MountingHole_2.1mm, MountingHole:MountingHole_2.1mm, F.Cu at (127.8, 99.1)
- added REF**: MountingHole_2.1mm, MountingHole:MountingHole_2.1mm, F.Cu at (156.3, 99.1)
- moved GND 2.32 mm to (128.7, 95.4)
- moved MOSI 2.32 mm to (128.7, 81.5)
- moved SCK 2.32 mm to (128.7, 79.1)
- moved 3.3 2.32 mm to (128.7, 90.8)
- moved CS 2.32 mm to (128.7, 84.0)
- moved SCL 2.32 mm to (128.7, 86.3)
- moved SDA 2.32 mm to (128.7, 88.5)
- moved VCC 2.32 mm to (128.7, 93.1)
- moved R4 0.13 mm to (141.7, 93.4)
- moved LED1 0.05 mm to (147.9, 77.6)
Routing:
- net Net-(D1-Pad2): track 13.1 -> 2.16 mm
- net VCC: track 43.4 -> 36.7 mm
- net /SCK: track 27.0 -> 24.1 mm
- net /MOSI: track 25.1 -> 22.8 mm
- net /D3: track 45.5 -> 43.9 mm
- net /D4: track 16.5 -> 17.6 mm
- net /CS: track 25.8 -> 26.8 mm
- net GND: track 67.1 -> 68.0 mm
- net /D2: track 39.0 -> 38.2 mm
- net 3.3V: track 56.3 -> 55.6 mm, vias 10 -> 9
Other:
- outline, holes or cut-outs redrawn

Commit message: rev 0.2
Parts:
- removed 3.3V: TestPoint_THTPad_2.0x2.0mm_Drill1.0mm, TestPoint:TestPoint_THTPad_2.0x2.0mm_Drill1.0mm
Changed lines of the file:
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@@
     (tracks 508)
     (zones 0)
-    (modules 52)
+    (modules 51)
     (nets 49)
   )
@@
       (rotate (xyz 0 0 0))
     )
-  )
-  (module TestPoint:TestPoint_THTPad_2.0x2.0mm_Drill1.0mm (layer F.Cu)
-    (at 145.4404 77.7494)
-    (descr "THT rectangular pad as test Point, square 2.0mm_Drill1.0mm  side length, hole diameter 1.0mm")
-    (tags "test point THT pad rectangle square")
-    (attr virtual)
-    (fp_text reference 3.3V (at -0.508 -1.7272) (layer F.SilkS)
-      (effects (font (size 0.5 0.5) (thickness 0.125)))
-    )
-    (fp_text value TestPoint_THTPad_2.0x2.0mm_Drill1.0mm (at 0 2.05) (layer F.Fab)
-      (effects (font (size 1 1) (thickness 0.15)))
-    )
-    (fp_line (start 1.5 1.5) (end -1.5 1.5) (layer F.CrtYd) (width 0.05))
-    (fp_line (start 1.5 1.5) (end 1.5 -1.5) (layer F.CrtYd) (width 0.05))
-    (fp_line (start -1.5 -1.5) (end -1.5 1.5) (layer F.CrtYd) (width 0.05))
-    (fp_line (start -1.5 -1.5) (end 1.5 -1.5) (layer F.CrtYd) (width 0.05))
-    (fp_line (start -1.2 1.2) (end -1.2 -1.2) (layer F.SilkS) (width 0.12))
-    (fp_line (start 1.2 1.2) (end -1.2 1.2) (layer F.SilkS) (width 0.12))
-    (fp_line (start 1.2 -1.2) (end 1.2 1.2) (layer F.SilkS) (width 0.12))
-    (fp_line (start -1.2 -1.2) (end 1.2 -1.2) (layer F.SilkS) (width 0.12))
-    (fp_text user %R (at 0 -2) (layer F.Fab)
-      (effects (font (size 1 1) (thickness 0.15)))
-    )
-    (pad 1 thru_hole rect (at 0 0) (size 2 2) (drill 1) (layers *.Cu *.Mask)
-      (net 1 3.3V))
   )
   (module Package_QFP:TQFP-44_10x10mm_P0.8mm (layer F.Cu)
@@
   (segment (start 149.098 90.17) (end 149.7486 90.17) (width 0.4) (layer F.Cu) (net 2))
   (via (at 143.9164 90.2208) (size 0.6) (drill 0.3) (layers F.Cu B.Cu) (net 2))
-  (segment (start 143.9164 90.2208) (end 144.616401 89.520799) (width 0.4) (layer F.Cu) (net 2))
-  (segment (start 148.336 90.17) (end 149.098 90.17) (width 0.4) (layer F.Cu) (net 2))
-  (segment (start 147.686799 89.520799) (end 148.336 90.17) (width 0.4) (layer F.Cu) (net 2))
-  (segment (start 144.616401 89.520799) (end 147.686799 89.520799) (width 0.4) (layer F.Cu) (net 2))
   (segment (start 141.4781 76.835) (end 141.5288 76.8857) (width 0.4) (layer F.Cu) (net 2))
   (segment (start 136.8806 76.68768) (end 136.86028 76.708) (width 0.4) (layer F.Cu) (net 2))
@@
   (segment (start 148.5647 94.1578) (end 148.3615 93.9546) (width 0.4) (layer F.Cu) (net 2))
   (segment (start 149.2758 94.1578) (end 148.5647 94.1578) (width 0.4) (layer F.Cu) (net 2))
+  (segment (start 143.9164 90.2208) (end 144.616401 89.520799) (width 0.4) (layer F.Cu) (net 2))
+  (segment (start 148.569998 89.7128) (end 149.027198 90.17) (width 0.4) (layer F.Cu) (net 2))
+  (segment (start 144.616401 89.520799) (end 148.347199 89.520799) (width 0.4) (layer F.Cu) (net 2))
+  (segment (start 148.347199 89.520799) (end 148.5392 89.7128) (width 0.4) (layer F.Cu) (net 2))
+  (segment (start 149.027198 90.17) (end 149.2504 90.17) (width 0.4) (layer F.Cu) (net 2))
+  (segment (start 148.5392 89.7128) (end 148.569998 89.7128) (width 0.4) (layer F.Cu) (net 2))
   (segment (start 146.684494 93.9546) (end 146.7865 93.9546) (width 0.25) (layer F.Cu) (net 3) (status 30))
   (segment (start 145.5039 92.672) (end 145.5039 91.5647) (width 0.25) (layer F.Cu) (net 3) (status 20))
@@
   (segment (start 131.9784 93.8315) (end 132.334 93.4759) (width 0.4) (layer F.Cu) (net 7))
   (segment (start 132.0546 93.7553) (end 132.334 93.4759) (width 0.4) (layer F.Cu) (net 7))
-  (segment (start 141.873201 84.723201) (end 140.953901 83.803901) (width 0.4) (layer F.Cu) (net 7))
-  (segment (start 140.748902 82.6647) (end 139.8039 82.6647) (width 0.4) (layer F.Cu) (net 7))
-  (segment (start 140.953901 82.869699) (end 140.748902 82.6647) (width 0.4) (layer F.Cu) (net 7))
-  (segment (start 140.953901 83.803901) (end 140.953901 82.869699) (width 0.4) (layer F.Cu) (net 7))
-  (segment (start 139.804 86.6648) (end 139.8039 86.6647) (width 0.4) (layer F.Cu) (net 7))
-  (segment (start 141.1732 86.6648) (end 139.804 86.6648) (width 0.4) (layer F.Cu) (net 7))
-  (segment (start 141.873201 85.964799) (end 141.873201 84.723201) (width 0.4) (layer F.Cu) (net 7))
-  (segment (start 141.1732 86.6648) (end 141.873201 85.964799) (width 0.4) (layer F.Cu) (net 7))
   (segment (start 134.583389 88.733506) (end 134.583389 93.102211) (width 0.4) (layer F.Cu) (net 7))
   (segment (start 133.577998 87.728115) (end 134.583389 88.733506) (width 0.4) (layer F.Cu) (net 7))
@@
   (segment (start 136.25771 93.48411) (end 136.71296 93.93936) (width 0.4) (layer F.Cu) (net 7))
   (segment (start 134.88611 93.48411) (end 136.25771 93.48411) (width 0.4) (layer F.Cu) (net 7))
+  (segment (start 139.804 86.6648) (end 139.8039 86.6647) (width 0.4) (layer F.Cu) (net 7))
+  (segment (start 140.861424 82.6647) (end 139.8039 82.6647) (width 0.4) (layer F.Cu) (net 7))
+  (segment (start 141.873201 83.676477) (end 140.861424 82.6647) (width 0.4) (layer F.Cu) (net 7))
+  (segment (start 140.7415 86.6647) (end 141.873201 85.532999) (width 0.4) (layer F.Cu) (net 7))
+  (segment (start 141.873201 85.532999) (end 141.873201 83.676477) (width 0.4) (layer F.Cu) (net 7))
+  (segment (start 139.8039 86.6647) (end 140.7415 86.6647) (width 0.4) (layer F.Cu) (net 7))
   (segment (start 133.7819 82.1309) (end 133.8707 82.1309) (width 0.25) (layer F.Cu) (net 8))
   (segment (start 133.7692 82.1563) (end 133.7692 81.9276) (width 0.25) (layer F.Cu) (net 8))
