File: Hardware/Kicad Project/ArduinoProMicroUSB/ArduinoProMicroUSB.kicad_pcb (KiCad board)
At the start: 4 copper layers, 31.1 x 26 mm, 51 parts, among them J3 Display FPC, Q1 MMBT3904, U1 RV-3028-C7, U2 MIC5219, U3 USB-AB, U5 ATMEGA32U4QFN, Y1 16MHz

Commit message: rev 0.3
Changed lines of the file:
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@@
     (35 F.Paste user hide)
     (36 B.SilkS user hide)
-    (37 F.SilkS user)
+    (37 F.SilkS user hide)
     (38 B.Mask user hide)
     (39 F.Mask user hide)
@@
   )
   (setup
-    (last_trace_width 0.4)
+    (last_trace_width 0.25)
     (user_trace_width 0.15)
     (user_trace_width 0.2)
@@
       (effects (font (size 1 1) (thickness 0.15)))
     )
-    (fp_text user %R (at 8.001 -1.7145) (layer F.Fab)
-      (effects (font (size 1 1) (thickness 0.15)))
-    )
     (fp_circle (center 0 0) (end 1.05 0) (layer Cmts.User) (width 0.15))
     (fp_circle (center 0 0) (end 1.3 0) (layer F.CrtYd) (width 0.05))
+    (fp_text user %R (at 8.001 -1.7145) (layer F.Fab)
+      (effects (font (size 1 1) (thickness 0.15)))
+    )
     (pad "" np_thru_hole circle (at 0 0) (size 1.3 1.3) (drill 1.05) (layers *.Cu *.Mask))
   )
@@
       (effects (font (size 1 1) (thickness 0.15)))
     )
+    (fp_line (start 1.48 0.73) (end -1.48 0.73) (layer F.CrtYd) (width 0.05))
+    (fp_line (start 1.48 -0.73) (end 1.48 0.73) (layer F.CrtYd) (width 0.05))
+    (fp_line (start -1.48 -0.73) (end 1.48 -0.73) (layer F.CrtYd) (width 0.05))
+    (fp_line (start -1.48 0.73) (end -1.48 -0.73) (layer F.CrtYd) (width 0.05))
+    (fp_line (start -0.162779 0.51) (end 0.162779 0.51) (layer F.SilkS) (width 0.12))
+    (fp_line (start -0.162779 -0.51) (end 0.162779 -0.51) (layer F.SilkS) (width 0.12))
+    (fp_line (start 0.8 0.4) (end -0.8 0.4) (layer F.Fab) (width 0.1))
+    (fp_line (start 0.8 -0.4) (end 0.8 0.4) (layer F.Fab) (width 0.1))
+    (fp_line (start -0.8 -0.4) (end 0.8 -0.4) (layer F.Fab) (width 0.1))
+    (fp_line (start -0.8 0.4) (end -0.8 -0.4) (layer F.Fab) (width 0.1))
     (fp_text user %R (at 0 0 90) (layer F.Fab)
       (effects (font (size 0.4 0.4) (thickness 0.06)))
     )
-    (fp_line (start 1.48 0.73) (end -1.48 0.73) (layer F.CrtYd) (width 0.05))
-    (fp_line (start 1.48 -0.73) (end 1.48 0.73) (layer F.CrtYd) (width 0.05))
-    (fp_line (start -1.48 -0.73) (end 1.48 -0.73) (layer F.CrtYd) (width 0.05))
-    (fp_line (start -1.48 0.73) (end -1.48 -0.73) (layer F.CrtYd) (width 0.05))
-    (fp_line (start -0.162779 0.51) (end 0.162779 0.51) (layer F.SilkS) (width 0.12))
-    (fp_line (start -0.162779 -0.51) (end 0.162779 -0.51) (layer F.SilkS) (width 0.12))
-    (fp_line (start 0.8 0.4) (end -0.8 0.4) (layer F.Fab) (width 0.1))
-    (fp_line (start 0.8 -0.4) (end 0.8 0.4) (layer F.Fab) (width 0.1))
-    (fp_line (start -0.8 -0.4) (end 0.8 -0.4) (layer F.Fab) (width 0.1))
-    (fp_line (start -0.8 0.4) (end -0.8 -0.4) (layer F.Fab) (width 0.1))
     (pad 1 smd roundrect (at -0.7875 0 90) (size 0.875 0.95) (layers F.Cu F.Paste F.Mask) (roundrect_rratio 0.25)
       (net 17 "Net-(Q1-Pad1)"))
@@
   (segment (start 149.7486 90.17) (end 150.0539 89.8647) (width 0.4) (layer F.Cu) (net 2))
   (segment (start 150.0539 89.8647) (end 151.2039 89.8647) (width 0.4) (layer F.Cu) (net 2))
-  (segment (start 149.098 90.17) (end 149.7486 90.17) (width 0.4) (layer F.Cu) (net 2))
   (via (at 143.9164 90.2208) (size 0.6) (drill 0.3) (layers F.Cu B.Cu) (net 2))
   (segment (start 141.4781 76.835) (end 141.5288 76.8857) (width 0.4) (layer F.Cu) (net 2))
@@
   (segment (start 148.5647 94.1578) (end 148.3615 93.9546) (width 0.4) (layer F.Cu) (net 2))
   (segment (start 149.2758 94.1578) (end 148.5647 94.1578) (width 0.4) (layer F.Cu) (net 2))
-  (segment (start 143.9164 90.2208) (end 144.616401 89.520799) (width 0.4) (layer F.Cu) (net 2))
-  (segment (start 148.569998 89.7128) (end 149.027198 90.17) (width 0.4) (layer F.Cu) (net 2))
-  (segment (start 144.616401 89.520799) (end 148.347199 89.520799) (width 0.4) (layer F.Cu) (net 2))
-  (segment (start 148.347199 89.520799) (end 148.5392 89.7128) (width 0.4) (layer F.Cu) (net 2))
-  (segment (start 149.027198 90.17) (end 149.2504 90.17) (width 0.4) (layer F.Cu) (net 2))
-  (segment (start 148.5392 89.7128) (end 148.569998 89.7128) (width 0.4) (layer F.Cu) (net 2))
+  (segment (start 143.9164 90.2208) (end 145.3134 90.2208) (width 0.25) (layer F.Cu) (net 2))
+  (segment (start 146.629401 89.595799) (end 147.1422 90.108598) (width 0.25) (layer F.Cu) (net 2))
+  (segment (start 145.3134 90.2208) (end 145.938401 89.595799) (width 0.25) (layer F.Cu) (net 2))
+  (segment (start 145.938401 89.595799) (end 146.629401 89.595799) (width 0.25) (layer F.Cu) (net 2))
+  (segment (start 149.188998 90.108598) (end 149.2504 90.17) (width 0.25) (layer F.Cu) (net 2))
+  (segment (start 147.1422 90.108598) (end 149.188998 90.108598) (width 0.25) (layer F.Cu) (net 2))
+  (segment (start 149.2504 90.17) (end 149.7486 90.17) (width 0.25) (layer F.Cu) (net 2))
   (segment (start 146.684494 93.9546) (end 146.7865 93.9546) (width 0.25) (layer F.Cu) (net 3) (status 30))
   (segment (start 145.5039 92.672) (end 145.5039 91.5647) (width 0.25) (layer F.Cu) (net 3) (status 20))
@@
   (segment (start 134.88611 93.48411) (end 136.25771 93.48411) (width 0.4) (layer F.Cu) (net 7))
   (segment (start 139.804 86.6648) (end 139.8039 86.6647) (width 0.4) (layer F.Cu) (net 7))
-  (segment (start 140.861424 82.6647) (end 139.8039 82.6647) (width 0.4) (layer F.Cu) (net 7))
-  (segment (start 141.873201 83.676477) (end 140.861424 82.6647) (width 0.4) (layer F.Cu) (net 7))
-  (segment (start 140.7415 86.6647) (end 141.873201 85.532999) (width 0.4) (layer F.Cu) (net 7))
-  (segment (start 141.873201 85.532999) (end 141.873201 83.676477) (width 0.4) (layer F.Cu) (net 7))
-  (segment (start 139.8039 86.6647) (end 140.7415 86.6647) (width 0.4) (layer F.Cu) (net 7))
+  (segment (start 140.613902 86.6647) (end 139.8039 86.6647) (width 0.25) (layer F.Cu) (net 7))
+  (segment (start 141.798201 85.480401) (end 140.613902 86.6647) (width 0.25) (layer F.Cu) (net 7))
+  (segment (start 141.798201 83.659001) (end 141.798201 85.480401) (width 0.25) (layer F.Cu) (net 7))
+  (segment (start 140.8039 82.6647) (end 141.798201 83.659001) (width 0.25) (layer F.Cu) (net 7))
+  (segment (start 139.8039 82.6647) (end 140.8039 82.6647) (width 0.25) (layer F.Cu) (net 7))
   (segment (start 133.7819 82.1309) (end 133.8707 82.1309) (width 0.25) (layer F.Cu) (net 8))
   (segment (start 133.7692 82.1563) (end 133.7692 81.9276) (width 0.25) (layer F.Cu) (net 8))

Commit message: updated schematic
Changed lines of the file:
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@@
   (page A4)
   (layers
-    (0 F.Cu signal)
-    (1 In1.Cu signal)
-    (2 In2.Cu signal)
-    (31 B.Cu signal)
+    (0 F.Cu signal hide)
+    (1 In1.Cu signal hide)
+    (2 In2.Cu signal hide)
+    (31 B.Cu signal hide)
     (32 B.Adhes user hide)
     (33 F.Adhes user hide)
     (34 B.Paste user hide)
-    (35 F.Paste user hide)
+    (35 F.Paste user)
     (36 B.SilkS user hide)
-    (37 F.SilkS user hide)
+    (37 F.SilkS user)
     (38 B.Mask user hide)
     (39 F.Mask user hide)
@@
   (gr_arc (start 156.3116 99.1362) (end 156.3116 100.4316) (angle -91.10170612) (layer Edge.Cuts) (width 0.05))
   (gr_arc (start 156.2735 75.7555) (end 157.606999 75.692001) (angle -87.27368901) (layer Edge.Cuts) (width 0.05))
-  (gr_line (start 127.838699 100.456989) (end 156.3116 100.4316) (layer Edge.Cuts) (width 0.05))
+  (gr_line (start 127.838699 100.457) (end 156.3116 100.4316) (layer Edge.Cuts) (width 0.05))
   (gr_line (start 126.493057 75.743794) (end 126.492001 99.110801) (layer Edge.Cuts) (width 0.05))
   (gr_line (start 156.2735 74.422) (end 127.762 74.422) (layer Edge.Cuts) (width 0.05))

Commit message: changelog
Connections:
- U3 pad SHLD: (no net) -> GND
Routing:
- net GND: track 68.0 -> 78.6 mm

Commit message: rev 0.4
Parts:
- removed 3.3, CS, GND, MOSI, SCK, SCL, SDA, VCC: TestPoint_THTPad_1.5x1.5mm_Drill0.7mm, TestPoint:TestPoint_THTPad_1.5x1.5mm_Drill0.7mm
- removed C13: 470pF, Capacitor_SMD:C_0603_1608Metric
- removed C3: 1uF, Capacitor_SMD:C_0603_1608Metric
- removed C4: 0.1uF, Capacitor_SMD:C_0603_1608Metric
- removed C8: 10nF, Capacitor_SMD:C_0603_1608Metric
- removed D1: DIODESOD, Diode_SMD:D_SOD-123
- removed F1: 500mA, Fuse:Fuse_1812_4532Metric
- removed LED1: Red, Diode_SMD:D_0603_1608Metric
- removed REF** (x4): MountingHole_2.1mm, MountingHole:MountingHole_2.1mm
- removed RN2: R_Pack04, Resistor_SMD:R_Array_Concave_4x0603
- removed U2: MIC5219, Downloads:SOT23-5
- added C14: 100pF, Capacitor_SMD:C_0603_1608Metric, F.Cu at (105.3, 74.8)
- added C15: 100pF, Capacitor_SMD:C_0603_1608Metric, F.Cu at (105.3, 73.3)
- added C16: 100pF, Capacitor_SMD:C_0603_1608Metric, F.Cu at (105.3, 68.5)
- added C17: 4.7uF, Capacitor_SMD:C_0603_1608Metric, F.Cu at (87.9, 76.6)
- added C18: 10uF, Capacitor_SMD:C_0603_1608Metric, F.Cu at (87.9, 84.5)
- added C9: 100pF, Capacitor_SMD:C_0603_1608Metric, F.Cu at (87.1, 66.8)
- added D4: PRTR5V0U2X,215, Downloads:SOT143B, F.Cu at (84.5, 70.2)
- added J1: Conn2, Downloads:1X02, F.Cu at (66.0, 69.8)
- added L1: 2.2uH, Inductor_SMD:L_0603_1608Metric, F.Cu at (87.9, 82.8)
- added R10: 6k, Resistor_SMD:R_0603_1608Metric, F.Cu at (85.5, 79.0)
- added R16: 267k, Resistor_SMD:R_0603_1608Metric, F.Cu at (85.5, 82.2)
- added SW1: SW_Push, Downloads:FSMRACD, F.Cu at (77.5, 89.3)
- added SW2: SW_Push, Downloads:FSMRACD, F.Cu at (84.8, 63.8)
- added SW3: SW_Push, Downloads:FSMRACD, F.Cu at (103.1, 89.2)
- added SW4: SW_Push, Downloads:FSMRACD, F.Cu at (109.9, 63.8)
- added TP1: TestPoint, TestPoint:TestPoint_Pad_1.0x1.0mm, B.Cu at (106.9, 78.5)
- added TP2: TestPoint, TestPoint:TestPoint_Pad_1.0x1.0mm, B.Cu at (106.9, 82.9)
- added TP3: TestPoint, TestPoint:TestPoint_Pad_1.0x1.0mm, B.Cu at (106.8, 76.3)
- added TP4: TestPoint, TestPoint:TestPoint_Pad_1.0x1.0mm, B.Cu at (106.9, 69.8)
- added TP5: TestPoint, TestPoint:TestPoint_Pad_1.0x1.0mm, B.Cu at (106.9, 80.6)
- added TP6: TestPoint, TestPoint:TestPoint_Pad_1.0x1.0mm, B.Cu at (106.9, 72.0)
- added TP7: TestPoint, TestPoint:TestPoint_Pad_1.0x1.0mm, B.Cu at (106.8, 74.2)
- added U4: TPS62840DLCR, Downloads:SON50P200X150X100-8N, F.Cu at (87.6, 80.5)
- C1, C2: value 10uF -> 100nF; footprint Capacitors:EIA3216 -> Capacitor_SMD:C_0603_1608Metric
- J3: value Display FPC -> FPC
- R2: value 1K -> 6k
- R9: value 10K -> R
- U3: footprint Connectors:USB-AB-MICRO-SMD -> Downloads:USB-AB-MICRO-SMD
- moved C7 70.3 mm to (85.5, 85.3), turned to 270 degrees
- moved R3 69.3 mm to (87.1, 86.9)
- moved R1 66.3 mm to (88.6, 86.9)
- moved U3 63.2 mm to (78.7, 75.8), turned to 0 degrees
- moved R8 62.6 mm to (90.2, 84.6), turned to 270 degrees
- moved R2 61.5 mm to (87.9, 78.2), turned to 0 degrees
- moved Q1 60.0 mm to (92.4, 85.6), turned to 0 degrees
- moved R7 54.0 mm to (87.9, 71.1), turned to 180 degrees
- moved D3 53.9 mm to (85.5, 73.6), turned to 90 degrees
- moved R11 53.4 mm to (84.7, 76.6)
- moved R5 53.3 mm to (87.9, 69.5), turned to 180 degrees
- moved U1 53.2 mm to (102.2, 84.1), turned to 0 degrees
- moved R6 51.7 mm to (102.0, 81.3), turned to 0 degrees
- moved C12 51.5 mm to (87.1, 73.7), turned to 90 degrees
- moved R15 51.4 mm to (105.3, 70.1)
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Connections:
- net /CS renamed /MISO
- C11 pad 2: Net-(C11-Pad2) -> 3.3V
- R2 pad 2: 3.3V -> GND
- R9 pad 1: Net-(R9-Pad1) -> 3.3V
- R9 pad 2: GND -> Net-(R9-Pad2)
- U1 pad 1: /32K -> Net-(U1-Pad1)
- U1 pad 6: Net-(R9-Pad1) -> 3.3V
- U1 pad 8: /D12 -> Net-(R9-Pad2)
- U3 pad SHLD: GND -> (no net)
- U5 pad 2: VCC -> Net-(U5-Pad2)
- U5 pad 28: /BTN2 -> /BTN3
- U5 pad 29: /BTN3 -> /BTN4
- U5 pad 30: /BTN4 -> /BTN2
- U5 pad 32: /32K -> /D13
- U5 pad 6: Net-(C11-Pad2) -> 3.3V
Routing:
- net /D3: track 43.9 -> 7.63 mm, vias 1 -> 2
- net /D2: track 38.2 -> 11.5 mm
- net /MISO: track 26.8 -> 1.42 mm
- net /D5: track 24.2 -> 0.00 mm, vias 1 -> 0
- net /LEDK: track 19.9 -> 0.00 mm
- net /SCK: track 24.1 -> 4.46 mm
- net /32K: track 18.3 -> 0.00 mm, vias 2 -> 0
- net /MOSI: track 22.8 -> 4.85 mm
- net /D4: track 17.6 -> 0.00 mm, vias 1 -> 0
- net /D12: track 15.9 -> 0.00 mm, vias 2 -> 0
- net GND: track 78.6 -> 64.1 mm, vias 19 -> 2
- net VCC: track 36.3 -> 23.6 mm
- net /RAW: track 10.9 -> 0.00 mm
- net Net-(R7-Pad2): track 2.41 -> 11.2 mm
- net Net-(R5-Pad2): track 2.84 -> 11.0 mm
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- removed copper zone on In2.Cu, net 3.3V
- removed copper zone on In1.Cu, net GND
Other:
- board size 31.1 x 26 mm -> 34.7 x 24.8 mm

Commit message: working on pcb
Parts:
- removed TP1, TP2, TP3, TP4, TP5, TP6, TP7: TestPoint, TestPoint:TestPoint_Pad_1.0x1.0mm
- added GND: TestPoint, TestPoint:TestPoint_Pad_1.0x1.0mm, F.Cu at (106.4, 95.6)
- added MOSI: TestPoint, TestPoint:TestPoint_Pad_1.0x1.0mm, F.Cu at (102.2, 95.6)
- added REF**: MountingHole_2.1mm, MountingHole:MountingHole_2.1mm, F.Cu at (88.3, 73.0)
- added REF**: MountingHole_2.1mm, MountingHole:MountingHole_2.1mm, F.Cu at (88.3, 95.6)
- added REF**: MountingHole_2.1mm, MountingHole:MountingHole_2.1mm, F.Cu at (115.4, 95.6)
- added REF**: MountingHole_2.1mm, MountingHole:MountingHole_2.1mm, F.Cu at (115.4, 73.0)
- added SCK: TestPoint, TestPoint:TestPoint_Pad_1.0x1.0mm, F.Cu at (100.1, 95.6)
- added SCL: TestPoint, TestPoint:TestPoint_Pad_1.0x1.0mm, F.Cu at (105.2, 73.2)
- added SDA: TestPoint, TestPoint:TestPoint_Pad_1.0x1.0mm, F.Cu at (106.9, 73.2)
- added SS: TestPoint, TestPoint:TestPoint_Pad_1.0x1.0mm, F.Cu at (98.0, 95.6)
- added VCC: TestPoint, TestPoint:TestPoint_Pad_1.0x1.0mm, F.Cu at (104.3, 95.6)
- C1, C10, C11, C12, C14, C15, C16, C17, C18, C2, C5, C6, C7, C9: footprint Capacitor_SMD:C_0603_1608Metric -> Downloads:0603
- L1: footprint Inductor_SMD:L_0603_1608Metric -> Downloads:0603
- R1, R10, R11, R12, R13, R14, R15, R16, R2, R3, R4, R5, R6, R7, R8, R9: footprint Resistor_SMD:R_0603_1608Metric -> Downloads:0603
- SW1, SW2, SW3, SW4: footprint Downloads:FSMRACD -> Downloads:Panasonic-EVP-AKE31A-MFG
- U5: footprint Package_QFP:TQFP-44_10x10mm_P0.8mm -> Downloads:QFN50P700X700X100-45N
- moved SW1 34.2 mm to (111.1, 95.9), turned to 270 degrees
- moved J1 32.7 mm to (98.6, 72.8)
- moved D3 20.3 mm to (100.1, 87.6), turned to 270 degrees
- moved D4 18.9 mm to (100.9, 79.6)
- moved R11 18.4 mm to (101.0, 85.3)
- moved C12 17.0 mm to (101.0, 83.6), turned to 180 degrees
- moved R12 16.3 mm to (101.9, 76.4)
- moved C9 16.1 mm to (100.1, 76.4)
- moved C11 14.8 mm to (101.0, 81.9), turned to 0 degrees
- moved C10 14.6 mm to (104.8, 75.6)
- moved R7 13.6 mm to (97.7, 80.5)
- moved R5 13.5 mm to (97.7, 78.8)
- moved U5 12.8 mm to (107.3, 80.6)
- moved R10 12.7 mm to (95.4, 87.0), turned to 90 degrees
- moved U3 12.4 mm to (88.5, 83.4)
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Connections:
- J3 pad 8: /MISO -> /D12
Routing:
- net VCC: track 23.6 -> 65.4 mm, vias 0 -> 2
- net /D12: track 0.00 -> 40.9 mm, vias 0 -> 2
- net /BTN4: track 4.26 -> 43.5 mm
- net 3.3V: track 62.5 -> 96.9 mm, vias 0 -> 4
- net /SCK: track 4.46 -> 36.3 mm, vias 1 -> 2
- net /MOSI: track 4.85 -> 35.4 mm, vias 1 -> 2
- net /LEDK: track 0.00 -> 22.8 mm, vias 1 -> 2
- net /BTN3: track 4.68 -> 24.4 mm
- net /D4: track 0.00 -> 17.7 mm, vias 0 -> 1
- net /D5: track 0.00 -> 17.4 mm, vias 0 -> 2
- net Net-(R6-Pad1): track 2.21 -> 15.2 mm
- net /BTN1: track 4.89 -> 15.2 mm, vias 0 -> 1
- net /BTN2: track 5.02 -> 13.1 mm
- net Net-(R7-Pad2): track 11.2 -> 7.67 mm
- net /D11: track 18.5 -> 15.1 mm
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- added copper zone on B.Cu, net GND
Other:
- board size 34.7 x 24.8 mm -> 31 x 26.4 mm
- board text added: "+"
- board text added: "-"
- board text added: "1.0"
- board text added: "ADRIAN"
- board text added: "FLUDER"

Commit message: finishing hardware design
Parts:
- removed SCL, SDA: TestPoint, TestPoint:TestPoint_Pad_1.0x1.0mm
- moved R7 1.54 mm to (96.2, 80.3)
- moved D4 1.47 mm to (99.4, 79.5)
- moved R5 1.47 mm to (96.2, 78.8)
- moved R11 0.29 mm to (101.2, 85.2)
- moved C12 0.28 mm to (101.2, 83.6)
- moved R12 0.17 mm to (101.9, 76.2)
- moved C9 0.14 mm to (100.1, 76.3)
- moved L1 0.08 mm to (98.4, 84.3)
- moved C17 0.06 mm to (93.9, 82.8)
- moved R2 0.06 mm to (93.9, 86.1)
- moved R4 0.05 mm to (103.0, 86.8)
- renumbered SS to TP1, MOSI to TP2, SCK to TP3, GND to TP6, VCC to TP7
Routing:
- net GND: track 66.7 -> 112.8 mm, vias 13 -> 20
- net 3.3V: track 96.9 -> 109.6 mm
- net /LEDK: track 22.8 -> 30.9 mm
- net /D-: track 6.08 -> 7.78 mm
- net /D5: track 17.4 -> 18.9 mm
- net Net-(R7-Pad2): track 7.67 -> 6.21 mm
- net /D+: track 6.40 -> 7.69 mm
- net Net-(R5-Pad2): track 8.15 -> 6.89 mm
- net /SCK: track 36.3 -> 37.2 mm
- net /MOSI: track 35.4 -> 36.2 mm
- net Net-(R6-Pad1): track 15.2 -> 15.8 mm, vias 0 -> 2
- net VCC: track 65.4 -> 65.2 mm, vias 2 -> 3
- added copper zone on F.Cu, net GND

Commit message: updated pcb
Routing:
- removed copper zone on F.Cu, net GND
