File: Hardware/Kicad Project/Kicad_Smart_Watch/Kicad_Smart_Watch.sch (KiCad schematic (older format))
At the start: 53 parts, among them J1 Conn2, J3 FPC, Q1 MMBT3904, SW1 SW_Push, SW2 SW_Push, SW3 SW_Push, SW4 SW_Push, U1 RV-3028-C7, U3 USB-AB, U4 TPS62840DLCR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

Commit message: updated mcu board pcb
Parts:
- SW1, SW2, SW3, SW4: footprint Downloads:Panasonic-EVP-AKE31A-MFG -> Downloads:1X02
Changed lines of the file:
@@
 F 0 "SW4" H 9720 4765 50  0000 C CNN
 F 1 "SW_Push" H 9720 4540 50  0000 C CNN
-F 2 "Downloads:Panasonic-EVP-AKE31A-MFG" H 9720 4815 50  0001 C CNN
+F 2 "Downloads:1X02" H 9720 4815 50  0001 C CNN
 F 3 "~" H 9720 4815 50  0001 C CNN
 	1    9720 4615
@@
 F 0 "SW1" H 8650 4775 50  0000 C CNN
 F 1 "SW_Push" H 8650 4550 50  0000 C CNN
-F 2 "Downloads:Panasonic-EVP-AKE31A-MFG" H 8650 4825 50  0001 C CNN
+F 2 "Downloads:1X02" H 8650 4825 50  0001 C CNN
 F 3 "~" H 8650 4825 50  0001 C CNN
 	1    8650 4625
@@
 F 0 "SW2" H 8060 4790 50  0000 C CNN
 F 1 "SW_Push" H 8060 4540 50  0000 C CNN
-F 2 "Downloads:Panasonic-EVP-AKE31A-MFG" H 8060 4815 50  0001 C CNN
+F 2 "Downloads:1X02" H 8060 4815 50  0001 C CNN
 F 3 "~" H 8060 4815 50  0001 C CNN
 	1    8060 4615
@@
 F 0 "SW3" H 9185 4770 50  0000 C CNN
 F 1 "SW_Push" H 9185 4545 50  0000 C CNN
-F 2 "Downloads:Panasonic-EVP-AKE31A-MFG" H 9185 4820 50  0001 C CNN
+F 2 "Downloads:1X02" H 9185 4820 50  0001 C CNN
 F 3 "~" H 9185 4820 50  0001 C CNN
 	1    9185 4620

Commit message: update
Parts:
- removed C1: 100nF, Downloads:0603, symbol Device:C
- removed TP6, TP7: TestPoint, TestPoint:TestPoint_Pad_1.0x1.0mm, symbol Connector:TestPoint
- added C3, C4: 4.7uF, Downloads:0603, symbol Device:C
- added D1, D5: D_Schottky, Downloads:0603, symbol Device:D_Schottky
- added D6: LED, Downloads:0603, symbol Device:LED
- added Q2: MCP73831_2, Downloads:SON50P200X300X100-9N, symbol misc:MCP73831_2
- added R17: 2k, Downloads:0603, symbol Device:R
- added R18: 10k, Downloads:0603, symbol Device:R
- R9: value R -> 10k
- U1: symbol RV-3028-C7:RV-3028-C7 -> Kicad_Smart_Watch-rescue:RV-3028-C7-RV-3028-C7
- U3: footprint Downloads:USB-AB-MICRO-SMD -> Downloads:GCT_USB3155-XX-X_REVA
Connections:
- net D11: no longer U1.2 (~INT~)
- net GND: now also J1.1, C3.2, C4.2, D6.1 (K), Q2.6 (VSS), R17.2, R18.2; no longer J1.2
- net VCC: now also D1.1 (K), D5.1 (K); no longer C12.1, D4.4, U3.VBUS, U5.7 (VBUS)
- net at U1.6 (VBACKUP): now also R18.1
- net TXO renamed INT
- net INT: now also U1.2 (~INT~)
- new net: D6.2 (A), Q2.5 (STAT)
- new net: Q2.8 (PROG), R17.1
- new net BAT+: C4.1, D5.2 (A), J1.2, Q2.3 (VBAT), Q2.4 (VBAT)
- new net VBUS: C12.1, C3.1, D1.2 (A), D4.4, Q2.1 (VDD), Q2.2 (VDD), U3.VBUS, U5.7 (VBUS)
Other:
- note added: "Power and charging"
- note removed: "Battery"
- moved on the sheet: C10, C11, C12, C14, C15, C16, C17, C18, C2, C5, C6, C7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
